Commit message: ros1 config

File: src/hb_robot_description/urdf/hb_robot.urdf (robot description, URDF)
Before this commit: robot hb_robot, 15 links, 14 joints
Links:
- link robot_mount: geometry collision mesh filename=file:///root/ros_ws/jetson_repo/src/hb_robot_description/me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; visual mesh filename=file:///root/ros_ws/jetson_repo/src/hb_robot_description/me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
